Commit message: effort controller

File: src/skbot/skbot_description/urdf/skbot.xacro (robot description, xacro)
@@ -66,3 +66,19 @@
     <xacro:wheel lr="left" tY="1"/>
     <xacro:wheel lr="right" tY="-1"/>
+    <!-- Position Config -->
+    <ros2_control name="GazeboSystem" type="system">
+        <hardware>
+          <plugin>gazebo_ros2_control/GazeboSystem</plugin>
+        </hardware>
+        <joint name="right_wheel_hinge">
+          <command_interface name="effort"/>
+          <state_interface name="velocity"/>
+          <state_interface name="effort"/>
+        </joint>
+        <joint name="left_wheel_hinge">
+          <command_interface name="effort"/>
+          <state_interface name="velocity"/>
+          <state_interface name="effort"/>
+        </joint>
+      </ros2_control>
 </robot>

Commit message: diff

File: src/skbot/skbot_description/urdf/skbot.xacro (robot description, xacro)
@@ -18,4 +18,11 @@
     <xacro:include filename="$(find skbot_description)/urdf/materials.xacro" />
     <xacro:include filename="$(find skbot_description)/urdf/macros.xacro" />
+    <!-- <link name="base_link">
+    </link>
+    <joint name="base_link_joint" type="fixed">
+        <origin rpy="0 0 0" xyz="0 0 0"/>
+        <parent link="base_link"/>
+        <child link="chassis"/>
+      </joint> -->
     <link name="chassis">
         <pose> 0 0 0.1 0 0 0 </pose>
@@ -67,5 +74,5 @@
     <xacro:wheel lr="right" tY="-1"/>
     <!-- Position Config -->
-    <ros2_control name="GazeboSystem" type="system">
+    <!-- <ros2_control name="GazeboSystem" type="system">
         <hardware>
           <plugin>gazebo_ros2_control/GazeboSystem</plugin>
@@ -81,4 +88,4 @@
           <state_interface name="effort"/>
         </joint>
-      </ros2_control>
+      </ros2_control> -->
 </robot>

Commit message: camera and gazebo launch

File: src/skbot/skbot_description/urdf/skbot.xacro (robot description, xacro)
@@ -89,3 +89,30 @@
         </joint>
       </ros2_control> -->
+    <!-- Adding a Camera -->
+    <joint name="camera_base" type="fixed">
+        <parent link="chassis"/>
+        <child link="camera" />
+        <!--origin xyz="${chassisLength/2-cameraSize/2} 0 ${chassisHeight+wheelRadius}" rpy="0 0 0" /-->
+        <origin xyz=".2 0 0.1" rpy="0 0 0" />
+    </joint>
+    <link name="camera">
+        <collision>
+            <origin xyz="0 0 0" rpy="0 0 0"/>
+            <geometry>
+                <box size="${cameraSize} ${cameraSize} ${cameraSize}"/>
+            </geometry>
+        </collision>
+        <visual>
+            <origin xyz="0 0 0" rpy="0 0 0"/>
+            <geometry>
+                <box size="${cameraSize} ${cameraSize} ${cameraSize}"/>
+            </geometry>
+            <material name="blue"/>
+        </visual>
+        <inertial>
+            <mass value="${cameraMass}" />
+            <origin xyz="0 0 0" rpy="0 0 0"/>
+            <box_inertia m="${cameraMass}" x="${cameraSize}" y="${cameraSize}" z="${cameraSize}" />
+        </inertial>
+    </link>
 </robot>

Commit message: laser sensor

File: src/skbot/skbot_description/urdf/skbot.xacro (robot description, xacro)
@@ -116,3 +116,31 @@
         </inertial>
     </link>
+    <!-- Adding a Laser Scanner -->
+  <joint name="hokuyo_joint" type="fixed">
+    <axis xyz="0 1 0" />
+    <origin xyz="${chassisLength/2-0.005} 0 ${chassisHeight+wheelRadius}" rpy="0 0 0" />
+    <!--origin xyz=".15 0 .1" rpy="0 0 0"/-->
+    <parent link="chassis"/>
+    <child link="hokuyo"/>
+  </joint>
+  <!-- Hokuyo Laser -->
+  <link name="hokuyo">
+    <collision>
+      <origin xyz="0 0 0" rpy="0 0 0"/>
+      <geometry>
+        <box size="0.1 0.1 0.1"/>
+      </geometry>
+    </collision>
+    <visual>
+      <origin xyz="0 0 0" rpy="0 0 0"/>
+      <geometry>
+        <mesh filename="file://hokuyo.dae"/>
+      </geometry>
+    </visual>
+    <inertial>
+      <mass value="1e-5" />
+      <origin xyz="0 0 0" rpy="0 0 0"/>
+      <inertia ixx="1e-6" ixy="0" ixz="0" iyy="1e-6" iyz="0" izz="1e-6" />
+    </inertial>
+  </link>
 </robot>
