Commit message: bl0105

File: src/skbot/skbot_description/urdf/gazebo.xacro (robot description, xacro)
@@ -1,11 +1,11 @@
 <?xml version="1.0"?>
 <robot>
-  <gazebo reference="chassis">
-    <material>Gazebo/Orange</material>
+  <gazebo reference="base_link">
+    <material>Gazebo/Red</material>
   </gazebo>
-  <gazebo reference="caster_wheel">
-    <mu1>0.0</mu1>
-    <mu2>0.0</mu2>
-    <material>Gazebo/Red</material>
+  <gazebo reference="front_caster">
+    <mu1>0.01</mu1>
+    <mu2>0.01</mu2>
+    <material>Gazebo/White</material>
   </gazebo>
   <!-- <gazebo>
@@ -26,9 +26,9 @@
       </ros>
       <!-- wheels -->
-      <left_joint>left_wheel_hinge</left_joint>
-      <right_joint>right_wheel_hinge</right_joint>
+      <left_joint>drivewhl_l_joint</left_joint>
+      <right_joint>drivewhl_r_joint</right_joint>
       <!-- kinematics -->
-      <wheel_separation>${chassisWidth+wheelWidth}</wheel_separation>
-      <wheel_diameter>${2*wheelRadius}</wheel_diameter>
+      <wheel_separation>${base_width+wheel_width}</wheel_separation>
+      <wheel_diameter>${2*wheel_radius}</wheel_diameter>
       <!-- limits -->
       <max_wheel_torque>10</max_wheel_torque>

File: src/skbot/skbot_description/urdf/macros.xacro (robot description, xacro)
@@ -1,59 +1,23 @@
 <?xml version="1.0"?>
 <robot name="" xmlns:xacro="http://www.ros.org/wiki/xacro">
+  <xacro:macro name="box_inertia" params="m w h d">
+    <inertial>
+      <origin xyz="0 0 0" rpy="${pi/2} 0 ${pi/2}"/>
+      <mass value="${m}"/>
+      <inertia ixx="${(m/12) * (h*h + d*d)}" ixy="0.0" ixz="0.0" iyy="${(m/12) * (w*w + d*d)}" iyz="0.0" izz="${(m/12) * (w*w + h*h)}"/>
+    </inertial>
+  </xacro:macro>
   <xacro:macro name="cylinder_inertia" params="m r h">
-    <inertia  ixx="${m*(3*r*r+h*h)/12}" ixy = "0" ixz = "0"
-      iyy="${m*(3*r*r+h*h)/12}" iyz = "0"
-      izz="${m*r*r/2}"
-    />
+    <inertial>
+      <origin xyz="0 0 0" rpy="${pi/2} 0 0" />
+      <mass value="${m}"/>
+      <inertia ixx="${(m/12) * (3*r*r + h*h)}" ixy = "0" ixz = "0" iyy="${(m/12) * (3*r*r + h*h)}" iyz = "0" izz="${(m/2) * (r*r)}"/>
+    </inertial>
   </xacro:macro>
-    <xacro:macro name="box_inertia" params="m x y z">
-        <inertia  ixx="${m*(y*y+z*z)/12}" ixy = "0" ixz = "0"
-          iyy="${m*(x*x+z*z)/12}" iyz = "0"
-          izz="${m*(x*x+z*z)/12}"
-        />
-      </xacro:macro>
-      <xacro:macro name="sphere_inertia" params="m r">
-        <inertia  ixx="${2*m*r*r/5}" ixy = "0" ixz = "0"
-          iyy="${2*m*r*r/5}" iyz = "0"
-          izz="${2*m*r*r/5}"
-        />
-      </xacro:macro>
-      <xacro:macro name="wheel" params="lr tY">
-        <link name="${lr}_wheel">
-          <collision>
-            <origin xyz="0 0 0" rpy="0 ${PI/2} ${PI/2}" />
-            <geometry>
-              <cylinder length="${wheelWidth}" radius="${wheelRadius}"/>
-            </geometry>
-          </collision>
-          <visual>
-            <origin xyz="0 0 0" rpy="0 ${PI/2} ${PI/2}" />
-            <geometry>
-              <cylinder length="${wheelWidth}" radius="${wheelRadius}"/>
-            </geometry>
-            <material name="white"/>
-          </visual>
-          <inertial>
-            <origin xyz="0 0 0" rpy="0 ${PI/2} ${PI/2}" />
-            <mass value="${wheelMass}"/>
-            <xacro:cylinder_inertia m="${wheelMass}" r="${wheelRadius}" h="${wheelWidth}"/>
-          </inertial>
-        </link>
-        <gazebo reference="${lr}_wheel">
-          <mu1 value="1.0"/>
-          <mu2 value="1.0"/>
-          <kp  value="10000000.0" />
-          <kd  value="1.0" />
-          <fdir1 value="1 0 0"/>
-          <material>Gazebo/White</material>
-        </gazebo>
-        <joint name="${lr}_wheel_hinge" type="continuous">
-          <parent link="chassis"/>
-          <child link="${lr}_wheel"/>
-          <origin xyz="${-wheelPos+chassisLength} ${tY*wheelWidth/2+tY*chassisWidth/2} ${wheelRadius}" rpy="0 0 0" />
-          <axis xyz="0 1 0" rpy="0 0 0" />
-          <limit effort="100" velocity="100"/>
-          <joint_properties damping="0.0" friction="0.0"/>
-        </joint>
+  <xacro:macro name="sphere_inertia" params="m r">
+    <inertial>
+      <mass value="${m}"/>
+      <inertia ixx="${(2/5) * m * (r*r)}" ixy="0.0" ixz="0.0" iyy="${(2/5) * m * (r*r)}" iyz="0.0" izz="${(2/5) * m * (r*r)}"/>
+    </inertial>
   </xacro:macro>
 </robot>

File: src/skbot/skbot_description/urdf/materials.xacro (robot description, xacro)
@@ -17,3 +17,9 @@
         <color rgba="${255/255} ${108/255} ${10/255} 1.0"/>
     </material>
+    <material name="white">
+        <color rgba="${255/255} ${255/255} ${255/255} 1.0"/>
+      </material>
+      <material name="red">
+        <color rgba="${255/255} ${0/255} ${0/255} 1.0"/>
+      </material>
 </robot>

File: src/skbot/skbot_description/urdf/skbot.xacro (robot description, xacro)
@@ -1,146 +1,123 @@
-<?xml version="1.0"?>
-<robot name="skbot"
-    xmlns:xacro="http://www.ros.org/wiki/xacro">
-    <xacro:property name="PI" value="3.1415926535897931"/>
-    <xacro:property name="chassisHeight" value="0.1"/>
-    <xacro:property name="chassisLength" value="0.4"/>
-    <xacro:property name="chassisWidth" value="0.2"/>
-    <xacro:property name="chassisMass" value="50"/>
-    <xacro:property name="wheelWidth" value="0.05"/>
-    <xacro:property name="wheelRadius" value="0.1"/>
-    <xacro:property name="wheelPos" value="0.25"/>
-    <xacro:property name="wheelMass" value="5"/>
-    <xacro:property name="casterRadius" value="0.05"/>
-    <xacro:property name="casterMass" value="5"/>
-    <xacro:property name="cameraSize" value="0.05"/>
-    <xacro:property name="cameraMass" value="0.1"/>
-    <xacro:include filename="$(find skbot_description)/urdf/skbot.gazebo" />
-    <xacro:include filename="$(find skbot_description)/urdf/materials.xacro" />
-    <xacro:include filename="$(find skbot_description)/urdf/macros.xacro" />
-    <!-- <link name="base_link">
+<?xml version="1.0" ?>
+<robot name="basic_mobile_bot"
+  xmlns:xacro="http://ros.org/wiki/xacro">
+  <!-- #region properties-->
+  <xacro:property name="base_width" value="0.39"/>
+  <xacro:property name="base_length" value="0.70"/>
+  <xacro:property name="base_height" value="0.18"/>
+  <!-- Define the shape of the robot's two back wheels in meters -->
+  <xacro:property name="wheel_radius" value="0.14"/>
+  <xacro:property name="wheel_width" value="0.06"/>
+  <!-- x-axis points forward, y-axis points to left, z-axis points upwards -->
+  <!-- Define the gap between the wheel and chassis along y-axis in meters -->
+  <xacro:property name="wheel_ygap" value="0.035"/>
+  <!-- Position the wheels along the z-axis -->
+  <xacro:property name="wheel_zoff" value="0.05"/>
+  <!-- Position the wheels along the x-axis -->
+  <xacro:property name="wheel_xoff" value="0.221"/>
+  <!-- Position the caster wheel along the x-axis -->
+  <xacro:property name="caster_xoff" value="0.217"/>
+<!-- #endregion -->
+  <xacro:include filename="$(find skbot_description)/urdf/macros.xacro" />
+  <xacro:include filename="$(find skbot_description)/urdf/gazebo.xacro" />
+  <xacro:include filename="$(find skbot_description)/urdf/materials.xacro" />
+  <!-- ****************** ROBOT BASE FOOTPRINT ***************************  -->
+  <!-- Define the center of the main robot chassis projected on the ground -->
+  <link name="base_footprint"/>
+  <!-- The base footprint of the robot is located underneath the chassis -->
+  <joint name="base_joint" type="fixed">
+    <parent link="base_footprint"/>
+    <child link="base_link" />
+    <origin xyz="0.0 0.0 ${(wheel_radius+wheel_zoff)}" rpy="0 0 0"/>
+  </joint>
+  <!-- ********************** ROBOT BASE *********************************  -->
+  <link name="base_link">
+    <visual>
+      <origin xyz="0 0 -0.05" rpy="0 0 0"/>
+      <geometry>
+        <box size="${base_length} ${base_width} ${base_height}"/>
+        <!-- <mesh filename="package://basic_mobile_robot/meshes/robot_base.stl" /> -->
+      </geometry>
+      <material name="red"/>
+    </visual>
+    <collision>
+      <geometry>
+        <box size="${base_length} ${base_width} ${base_height}"/>
+      </geometry>
+    </collision>
+    <xacro:box_inertia m="40.0" w="${base_width}" d="${base_length}" h="${base_height}"/>
+  </link>
+  <!-- *********************** DRIVE WHEELS ******************************  -->
+  <xacro:macro name="wheel" params="prefix x_reflect y_reflect">
+    <link name="${prefix}_link">
+      <visual>
+        <origin xyz="0 0 0" rpy="1.5707963267949 0 0"/>
+        <geometry>
+          <cylinder radius="${wheel_radius}" length="${wheel_width}"/>
+        </geometry>
+        <material name="white"/>
+      </visual>
+      <collision>
+        <origin xyz="0 0 0" rpy="${pi/2} 0 0"/>
+        <geometry>
+          <cylinder radius="${wheel_radius}" length="${wheel_width}"/>
+        </geometry>
+      </collision>
+      <xacro:cylinder_inertia m="110.5" r="${wheel_radius}" h="${wheel_width}"/>
     </link>
-    <joint name="base_link_joint" type="fixed">
-        <origin rpy="0 0 0" xyz="0 0 0"/>
-        <parent link="base_link"/>
-        <child link="chassis"/>
-      </joint> -->
-    <link name="chassis">
-        <pose> 0 0 0.1 0 0 0 </pose>
-        <collision>
-            <origin xyz="0 0 ${wheelRadius}" rpy="0 0 0"/>
-            <geometry>
-                <box size="${chassisLength} ${chassisWidth} ${chassisHeight}"/>
-            </geometry>
-        </collision>
-        <visual>
-            <origin xyz="0 0 ${wheelRadius}" rpy="0 0 0"/>
-            <geometry>
-                <box size="${chassisLength} ${chassisWidth} ${chassisHeight}"/>
-            </geometry>
-            <material name="orange"/>
-        </visual>
-        <inertial>
-            <origin xyz="0 0 ${wheelRadius}" rpy="0 0 0"/>
-            <mass value="${chassisMass}"/>
-            <xacro:box_inertia m="${chassisMass}" x="${chassisLength}" y="${chassisWidth}" z="${chassisHeight}"/>
-        </inertial>
-    </link>
-    <joint name="fixed" type="fixed">
-        <parent link="chassis"/>
-        <child link="caster_wheel"/>
+    <!-- Connect the wheels to the base_link at the appropriate location, and
+         define a continuous joint to allow the wheels to freely rotate about
+         an axis -->
+    <joint name="${prefix}_joint" type="revolute">
+      <parent link="base_link"/>
+      <child link="${prefix}_link"/>
+      <origin xyz="${x_reflect*wheel_xoff} ${y_reflect*(base_width/2+wheel_ygap)} ${-wheel_zoff}" rpy="0 0 0"/>
+      <limit upper="3.1415" lower="-3.1415" effort="30" velocity="5.0"/>
+      <axis xyz="0 1 0"/>
     </joint>
-    <link name="caster_wheel">
-        <collision>
-            <origin xyz="${casterRadius-chassisLength/2} 0 ${casterRadius-chassisHeight+wheelRadius}" rpy="0 0 0"/>
-            <geometry>
-                <sphere radius="${casterRadius}"/>
-            </geometry>
-        </collision>
-        <visual>
-            <origin xyz="${casterRadius-chassisLength/2} 0 ${casterRadius-chassisHeight+wheelRadius}" rpy="0 0 0"/>
-            <geometry>
-                <sphere radius="${casterRadius}"/>
-            </geometry>
-            <material name="red"/>
-        </visual>
-        <inertial>
-            <origin xyz="${casterRadius-chassisLength/2} 0 ${casterRadius-chassisHeight+wheelRadius}" rpy="0 0 0"/>
-            <mass value="${casterMass}"/>
-            <xacro:sphere_inertia m="${casterMass}" r="${casterRadius}"/>
-        </inertial>
-    </link>
-    <!-- Adding Left and Right Wheels -->
-    <xacro:wheel lr="left" tY="1"/>
-    <xacro:wheel lr="right" tY="-1"/>
-    <!-- Position Config -->
-    <!-- <ros2_control name="GazeboSystem" type="system">
-        <hardware>
-          <plugin>gazebo_ros2_control/GazeboSystem</plugin>
-        </hardware>
-        <joint name="right_wheel_hinge">
-          <command_interface name="effort"/>
-          <state_interface name="velocity"/>
-          <state_interface name="effort"/>
-        </joint>
-        <joint name="left_wheel_hinge">
-          <command_interface name="effort"/>
-          <state_interface name="velocity"/>
-          <state_interface name="effort"/>
-        </joint>
-      </ros2_control> -->
-    <!-- Adding a Camera -->
-    <joint name="camera_base" type="fixed">
-        <parent link="chassis"/>
-        <child link="camera" />
-        <!--origin xyz="${chassisLength/2-cameraSize/2} 0 ${chassisHeight+wheelRadius}" rpy="0 0 0" /-->
-        <origin xyz=".2 0 0.1" rpy="0 0 0" />
-    </joint>
-    <link name="camera">
-        <collision>
-            <origin xyz="0 0 0" rpy="0 0 0"/>
-            <geometry>
-                <box size="${cameraSize} ${cameraSize} ${cameraSize}"/>
-            </geometry>
-        </collision>
-        <visual>
-            <origin xyz="0 0 0" rpy="0 0 0"/>
-            <geometry>
-                <box size="${cameraSize} ${cameraSize} ${cameraSize}"/>
-            </geometry>
-            <material name="blue"/>
-        </visual>
-        <inertial>
-            <mass value="${cameraMass}" />
-            <origin xyz="0 0 0" rpy="0 0 0"/>
-            <box_inertia m="${cameraMass}" x="${cameraSize}" y="${cameraSize}" z="${cameraSize}" />
-        </inertial>
-    </link>
-    <!-- Adding a Laser Scanner -->
-  <joint name="hokuyo_joint" type="fixed">
-    <axis xyz="0 1 0" />
-    <origin xyz="${chassisLength/2-0.005} 0 ${chassisHeight+wheelRadius}" rpy="0 0 0" />
-    <!--origin xyz=".15 0 .1" rpy="0 0 0"/-->
-    <parent link="chassis"/>
-    <child link="hokuyo"/>
-  </joint>
-  <!-- Hokuyo Laser -->
-  <link name="hokuyo">
+  </xacro:macro>
+  <!-- Instantiate two wheels using the macro we just made through the
+       xacro:wheel tags. We also define the parameters to have one wheel
+       on both sides at the back of our robot (i.e. x_reflect=-1). -->
+  <xacro:wheel prefix="drivewhl_l" x_reflect="-1" y_reflect="1" />
+  <xacro:wheel prefix="drivewhl_r" x_reflect="-1" y_reflect="-1" />
+  <!-- *********************** CASTER WHEEL ******************************  -->
+  <!-- We add a caster wheel. It will be modeled as sphere.
+       We define the wheel’s geometry, material and the joint to connect it to
+       base_link at the appropriate location. -->
+  <link name="front_caster">
+    <visual>
+      <geometry>
+        <sphere radius="${(wheel_radius+wheel_zoff-(base_height/2))}"/>
+      </geometry>
+      <material name="white"/>
+    </visual>
     <collision>
       <origin xyz="0 0 0" rpy="0 0 0"/>
       <geometry>
-        <box size="0.1 0.1 0.1"/>
+        <sphere radius="${(wheel_radius+wheel_zoff-(base_height/2))}"/>
       </geometry>
     </collision>
-    <visual>
-      <origin xyz="0 0 0" rpy="0 0 0"/>
-      <geometry>
-        <mesh filename="file://hokuyo.dae"/>
-      </geometry>
-    </visual>
-    <inertial>
-      <mass value="1e-5" />
-      <origin xyz="0 0 0" rpy="0 0 0"/>
-      <inertia ixx="1e-6" ixy="0" ixz="0" iyy="1e-6" iyz="0" izz="1e-6" />
-    </inertial>
+    <xacro:sphere_inertia m="10.05" r="${(wheel_radius+wheel_zoff-(base_height/2))}"/>
   </link>
+  <joint name="caster_joint" type="fixed">
+    <parent link="base_link"/>
+    <child link="front_caster"/>
+    <origin xyz="${caster_xoff} 0.0 ${-(base_height/2)}" rpy="0 0 0"/>
+  </joint>
+  <!-- *********************** IMU SETUP *********************************  -->
+  <!-- Each sensor must be attached to a link.                              -->
+  <joint name="imu_joint" type="fixed">
+    <parent link="base_link"/>
+    <child link="imu_link"/>
+    <origin xyz="-0.10 0 0.05" rpy="0 0 0"/>
+  </joint>
+  <link name="imu_link"/>
+  <!-- *********************** GPS SETUP **********************************  -->
+  <joint name="gps_joint" type="fixed">
+    <parent link="base_link"/>
+    <child link="gps_link"/>
+    <origin xyz="0.10 0 0.05" rpy="0 0 0"/>
+  </joint>
+  <link name="gps_link"/>
 </robot>
