Commit message: sdf schema
start to add xacro support to xml schema

File: src/skbot/skbot_gazebo/models/test/test.sdf.xacro (robot description, xacro)
@@ -1,5 +1,16 @@
 <?xml version="1.0"?>
-<sdf version="1.7">
+<sdf version="1.7" xmlns:xacro="http://www.ros.org/wiki/xacro">
+    <xacro:include filename="/home/user/dev_ws/vscode/sdf/templates/macros.xacro" />
+    <xacro:include filename="/home/user/dev_ws/vscode/sdf/templates/common.xacro" />
     <model name="test">
+        <link name="link_00">
+            <visual name="visual_00">
+                <geometry>
+                    <sphere>
+                        <radius>${PI}</radius>
+                    </sphere>
+                </geometry>
+            </visual>
+        </link>
     </model>
 </sdf>

Commit message: add xacro arg to schema

File: src/skbot/skbot_gazebo/models/test/test.sdf.xacro (robot description, xacro)
@@ -1,4 +1,6 @@
 <?xml version="1.0"?>
-<sdf version="1.7" xmlns:xacro="http://www.ros.org/wiki/xacro">
+<sdf version="1.7"
+    xmlns:xacro="http://www.ros.org/wiki/xacro">
+    <xacro:arg name="sphere" default="true" />
     <xacro:include filename="/home/user/dev_ws/vscode/sdf/templates/macros.xacro" />
     <xacro:include filename="/home/user/dev_ws/vscode/sdf/templates/common.xacro" />
@@ -7,7 +9,9 @@
             <visual name="visual_00">
                 <geometry>
-                    <sphere>
-                        <radius>${PI}</radius>
-                    </sphere>
+                    <xacro:if value="$(arg sphere)">
+                        <sphere>
+                            <radius>${PI}</radius>
+                        </sphere>
+                    </xacro:if>
                 </geometry>
             </visual>
